File: shield.kicad_pcb (KiCad board)
At the start: 2 copper layers, 26 parts, among them J1 USB_C_Receptacle_USB2.0_14P, U1 SRV05-4, U2 CH334F, U3 M24C02-WMN, Y1 12Mhz

Commit message: Add Uno shield
Parts:
- removed TP1, TP2, TP3, TP4: TestPoint, TestPoint:TestPoint_Pad_D1.5mm
- added A1: Arduino_UNO_R3, Module:Arduino_UNO_R3, F.Cu at (69.0, 107.1)
- added C10: 100nF, Capacitor_SMD:C_0402_1005Metric, F.Cu at (125.8, 95.8)
- added C4: 100nF, Capacitor_SMD:C_0402_1005Metric, F.Cu at (73.9, 93.9)
- added C5: 100nF, Capacitor_SMD:C_0402_1005Metric, F.Cu at (125.8, 85.9)
- added C6: 100nF, Capacitor_SMD:C_0402_1005Metric, F.Cu at (125.8, 87.9)
- added C7: 100nF, Capacitor_SMD:C_0402_1005Metric, F.Cu at (125.8, 89.8)
- added C8: 100nF, Capacitor_SMD:C_0402_1005Metric, F.Cu at (125.8, 91.8)
- added C9: 100nF, Capacitor_SMD:C_0402_1005Metric, F.Cu at (125.8, 93.8)
- added J2: USB_A, Connector_USB:USB_A_Receptacle_GCT_USB1046, F.Cu at (39.2, 92.6)
- added J3: USB_A, Connector_USB:USB_A_Receptacle_GCT_USB1046, F.Cu at (39.2, 76.7)
- added JP1: SolderJumper_2_Open, Jumper:SolderJumper-2_P1.3mm_Open_TrianglePad1.0x1.5mm, F.Cu at (111.9, 100.6)
- added R10: R, Resistor_SMD:R_0603_1608Metric_Pad0.98x0.95mm_HandSolder, F.Cu at (70.8, 84.7)
- added R11: 1R, Resistor_SMD:R_0402_1005Metric, F.Cu at (70.8, 86.7)
- added R12: 1K, Resistor_SMD:R_0402_1005Metric, F.Cu at (53.9, 85.6)
- added R13: 300K, Resistor_SMD:R_0603_1608Metric, F.Cu at (54.4, 83.3)
- added R14: R, Resistor_SMD:R_0603_1608Metric_Pad0.98x0.95mm_HandSolder, F.Cu at (54.6, 80.8)
- added R15: 1R, Resistor_SMD:R_0402_1005Metric, F.Cu at (53.9, 87.6)
- added R16: 470R, Resistor_SMD:R_0402_1005Metric, F.Cu at (84.6, 96.5)
- added R17: 470R, Resistor_SMD:R_0402_1005Metric, F.Cu at (111.2, 85.9)
- added R18: 470R, Resistor_SMD:R_0402_1005Metric, F.Cu at (111.2, 87.9)
- added R19: 470R, Resistor_SMD:R_0402_1005Metric, F.Cu at (111.2, 89.9)
- added R20: 470R, Resistor_SMD:R_0402_1005Metric, F.Cu at (111.2, 91.9)
- added R21: 470R, Resistor_SMD:R_0402_1005Metric, F.Cu at (111.2, 93.9)
- added R22: 470R, Resistor_SMD:R_0402_1005Metric, F.Cu at (111.2, 95.9)
- added R23: 470R, Resistor_SMD:R_0402_1005Metric, F.Cu at (111.2, 97.9)
- added R24: 470R, Resistor_SMD:R_0402_1005Metric, F.Cu at (114.1, 85.9)
- added R25: 470R, Resistor_SMD:R_0402_1005Metric, F.Cu at (114.1, 87.9)
- added R26: 470R, Resistor_SMD:R_0402_1005Metric, F.Cu at (114.1, 89.9)
- added R27: 470R, Resistor_SMD:R_0402_1005Metric, F.Cu at (114.1, 91.9)
- added R28: 470R, Resistor_SMD:R_0402_1005Metric, F.Cu at (114.1, 93.9)
- added R29: 470R, Resistor_SMD:R_0402_1005Metric, F.Cu at (114.1, 95.9)
- added R30: 470R, Resistor_SMD:R_0402_1005Metric, F.Cu at (114.1, 97.9)
- added R31: 470R, Resistor_SMD:R_0402_1005Metric, F.Cu at (117.0, 85.9)
- added R32: 470R, Resistor_SMD:R_0402_1005Metric, F.Cu at (117.0, 87.9)
- added R33: 470R, Resistor_SMD:R_0402_1005Metric, F.Cu at (117.0, 89.9)
- added R34: 470R, Resistor_SMD:R_0402_1005Metric, F.Cu at (117.0, 91.9)
- added R35: 470R, Resistor_SMD:R_0402_1005Metric, F.Cu at (117.0, 93.9)
- added R36: 470R, Resistor_SMD:R_0402_1005Metric, F.Cu at (117.0, 95.9)
- added R37: 470R, Resistor_SMD:R_0402_1005Metric, F.Cu at (117.0, 97.9)
- added R38: 470R, Resistor_SMD:R_0402_1005Metric, F.Cu at (120.0, 85.9)
- added R39: 470R, Resistor_SMD:R_0402_1005Metric, F.Cu at (120.0, 87.9)
- added R40: 470R, Resistor_SMD:R_0402_1005Metric, F.Cu at (120.0, 89.9)
- added R41: 470R, Resistor_SMD:R_0402_1005Metric, F.Cu at (120.0, 91.9)
- added R42: 470R, Resistor_SMD:R_0402_1005Metric, F.Cu at (120.0, 93.9)
- added R43: 470R, Resistor_SMD:R_0402_1005Metric, F.Cu at (120.0, 95.9)
- added R44: 470R, Resistor_SMD:R_0402_1005Metric, F.Cu at (120.0, 97.9)
- added R45: 470R, Resistor_SMD:R_0402_1005Metric, F.Cu at (122.9, 85.9)
- added R46: 470R, Resistor_SMD:R_0402_1005Metric, F.Cu at (122.9, 87.9)
- added R47: 470R, Resistor_SMD:R_0402_1005Metric, F.Cu at (122.9, 89.9)
- added R48: 470R, Resistor_SMD:R_0402_1005Metric, F.Cu at (122.9, 91.9)
- added R49: 470R, Resistor_SMD:R_0402_1005Metric, F.Cu at (122.9, 93.9)
- added R8: 1K, Resistor_SMD:R_0402_1005Metric, F.Cu at (70.6, 89.6)
- added R9: 300K, Resistor_SMD:R_0603_1608Metric, F.Cu at (66.4, 89.6)
- added U5: ~, Package_TO_SOT_SMD:SOT-23-6, F.Cu at (66.8, 86.1)
- added U6: ~, Package_TO_SOT_SMD:SOT-23-6, F.Cu at (67.4, 96.0)
- added U7: ~, Package_TO_SOT_SMD:SOT-23-6, F.Cu at (55.0, 77.4)
- U1: value SRV05-4 -> INA219AxDCN; footprint Package_TO_SOT_SMD:SOT-23-6 -> Package_TO_SOT_SMD:SOT-23-8
- U2: value CH334F -> SRV05-4; footprint Package_DFN_QFN:QFN-24-1EP_4x4mm_P0.5mm_EP2.7x2.7mm -> Package_TO_SOT_SMD:SOT-23-6
- U4: value ~ -> CH334F; footprint Package_TO_SOT_SMD:SOT-23-6 -> Package_DFN_QFN:QFN-24-1EP_4x4mm_P0.5mm_EP2.7x2.7mm
- moved J1 13.7 mm to (37.8, 63.4)
Connections:
- D1 pad 2: /USB/LED4/SDA -> /USB/I2C.SDA
- D2 pad 1: /USB/LED4/SDA -> /USB/I2C.SDA
- D3 pad 2: /USB/LED4/SDA -> /USB/I2C.SDA
- D4 pad 1: /USB/LED4/SDA -> /USB/I2C.SDA
- J1 pad A8: Net-(J1-SBU1) -> unconnected-(J1-SBU1-PadA8)
- J1 pad B8: Net-(J1-SBU2) -> unconnected-(J1-SBU2-PadB8)
- R3 pad 1: Net-(U4-ISET) -> Net-(U5-ISET)
- R7 pad 1: /USB/LED4/SDA -> /USB/I2C.SDA
- U1 pad 1: /USB/D+ -> unconnected-(U1-IN+-Pad1)
- U1 pad 2: GND -> unconnected-(U1-IN--Pad2)
- U1 pad 3: /USB/D- -> unconnected-(U1-GND-Pad3)
- U1 pad 5: /USB/VBUS -> unconnected-(U1-SCL-Pad5)
- U2 pad 1: /USB/~{FLAG} -> /USB/D+
- U2 pad 2: unconnected-(U2-NC-Pad2) -> GND
- U2 pad 3: Net-(U2-XO) -> /USB/D-
- U2 pad 4: Net-(U2-XI) -> unconnected-(U2-IO3-Pad4)
- U2 pad 5: /USB/USB4.D+ -> /USB/VBUS
- U2 pad 6: /USB/USB4.D- -> unconnected-(U2-IO4-Pad6)
- U3 pad 5: /USB/LED4/SDA -> /USB/I2C.SDA
- U4 pad 1: +5V -> /USB/~{FLAG}
- U4 pad 2: GND -> unconnected-(U4-NC-Pad2)
- U4 pad 3: /USB/~{FLAG} -> Net-(U4-XO)
- U4 pad 4: /USB/~{EN} -> Net-(U4-XI)
- U4 pad 5: Net-(U4-ISET) -> /USB/USB4.D+
- U4 pad 6: /USB/VBUS -> /USB/USB4.D-
- Y1 pad 1: Net-(U2-XI) -> Net-(U4-XI)
- Y1 pad 3: Net-(U2-XO) -> Net-(U4-XO)

Commit message: Start Layout
Parts:
- removed F1: 500mA, Fuse:Fuse_1206_3216Metric_Pad1.42x1.75mm_HandSolder
- added C11: 100nF, Capacitor_SMD:C_0402_1005Metric_Pad0.74x0.62mm_HandSolder, F.Cu at (61.0, 76.0)
- added C12: 100uF, Capacitor_SMD:C_1206_3216Metric, F.Cu at (183.2, 129.7)
- added C13: 100uF, Capacitor_SMD:C_1206_3216Metric, F.Cu at (257.3, 128.9)
- added C14: 15p, Capacitor_SMD:C_0402_1005Metric, F.Cu at (204.6, 110.7)
- added C15: 15p, Capacitor_SMD:C_0402_1005Metric, F.Cu at (114.0, 165.5)
- added C16: 15p, Capacitor_SMD:C_0402_1005Metric, F.Cu at (117.0, 165.5)
- added C17: 15p, Capacitor_SMD:C_0402_1005Metric, F.Cu at (204.6, 112.6)
- added C18: 4.7u, ProjectSpecific:C_0402_1005Metric_small_pads, F.Cu at (117.5, 148.0)
- added C19: 4.7u, ProjectSpecific:C_0402_1005Metric_small_pads, F.Cu at (117.5, 147.0)
- added C20: 100nF, Capacitor_SMD:C_0402_1005Metric, F.Cu at (122.0, 154.0)
- added C21: 4.7u, Capacitor_SMD:C_0402_1005Metric, F.Cu at (120.5, 147.5)
- added C22: 4.7u, Capacitor_SMD:C_0402_1005Metric, F.Cu at (115.0, 161.5)
- added C23: 100nF, Capacitor_SMD:C_0402_1005Metric, F.Cu at (107.0, 154.5)
- added C24: 100nF, Capacitor_SMD:C_0402_1005Metric, F.Cu at (122.0, 155.0)
- added C25: 100nF, Capacitor_SMD:C_0402_1005Metric, F.Cu at (112.0, 147.0)
- added C26: 100nF, Capacitor_SMD:C_0402_1005Metric, F.Cu at (107.0, 152.0)
- added C27: 100nF, Capacitor_SMD:C_0402_1005Metric, F.Cu at (107.0, 156.5)
- added C28: 100nF, Capacitor_SMD:C_0402_1005Metric, F.Cu at (112.0, 161.5)
- added C29: 100nF, Capacitor_SMD:C_0402_1005Metric, F.Cu at (113.5, 161.5)
- added C30: 100nF, Capacitor_SMD:C_0402_1005Metric, F.Cu at (122.0, 158.5)
- added C31: 100nF, Capacitor_SMD:C_0402_1005Metric, F.Cu at (122.0, 150.0)
- added C32: 100nF, Capacitor_SMD:C_0402_1005Metric, F.Cu at (114.5, 147.0)
- added C33: 10u, Capacitor_SMD:C_0805_2012Metric, F.Cu at (125.0, 146.0)
- added C34: 4.7u, ProjectSpecific:C_0402_1005Metric_small_pads, F.Cu at (204.6, 114.6)
- added C35: 4.7u, ProjectSpecific:C_0402_1005Metric_small_pads, F.Cu at (204.6, 116.6)
- added C36: 100nF, Capacitor_SMD:C_0402_1005Metric, F.Cu at (204.6, 118.5)
- added C37: 4.7u, Capacitor_SMD:C_0402_1005Metric, F.Cu at (204.6, 120.5)
- added C38: 4.7u, Capacitor_SMD:C_0402_1005Metric, F.Cu at (204.6, 122.5)
- added C39: 100nF, Capacitor_SMD:C_0402_1005Metric, F.Cu at (207.4, 110.7)
- added C40: 100nF, Capacitor_SMD:C_0402_1005Metric, F.Cu at (207.4, 112.6)
- added C41: 100nF, Capacitor_SMD:C_0402_1005Metric, F.Cu at (207.4, 114.6)
- added C42: 100nF, Capacitor_SMD:C_0402_1005Metric, F.Cu at (207.4, 116.6)
- added C43: 100nF, Capacitor_SMD:C_0402_1005Metric, F.Cu at (207.4, 118.5)
- added C44: 100nF, Capacitor_SMD:C_0402_1005Metric, F.Cu at (207.4, 120.5)
- added C45: 100nF, Capacitor_SMD:C_0402_1005Metric, F.Cu at (207.4, 122.5)
- added C46: 100nF, Capacitor_SMD:C_0402_1005Metric, F.Cu at (210.3, 110.7)
- added C47: 100nF, Capacitor_SMD:C_0402_1005Metric, F.Cu at (210.3, 112.6)
- added C48: 100nF, Capacitor_SMD:C_0402_1005Metric, F.Cu at (210.3, 114.6)
- added C49: 10u, Capacitor_SMD:C_0805_2012Metric, F.Cu at (221.8, 134.7)
- added C50: 100nF, Capacitor_SMD:C_0402_1005Metric, F.Cu at (112.0, 136.5)
- added C51: 100nF, Capacitor_SMD:C_0402_1005Metric, F.Cu at (210.3, 116.6)
- added C52: 100uF, Capacitor_SMD:C_1206_3216Metric, F.Cu at (252.8, 84.2)
- added C53: 100uF, Capacitor_SMD:C_1206_3216Metric, F.Cu at (183.2, 133.1)
- added C54: 100uF, Capacitor_SMD:C_1206_3216Metric, F.Cu at (183.2, 136.4)
- added C55: 1uF, Capacitor_SMD:C_0402_1005Metric, F.Cu at (173.0, 136.3)
- added C56: 100nF, Capacitor_SMD:C_0402_1005Metric, F.Cu at (173.0, 138.2)
- added C57: 22uF, Capacitor_SMD:C_0805_2012Metric, F.Cu at (178.1, 136.4)
- added D6: LED, LED_SMD:LED_0805_2012Metric, F.Cu at (263.4, 97.0)
- added D7: LED, LED_SMD:LED_0805_2012Metric, F.Cu at (269.9, 46.0)
- added F2: 1A, Fuse:Fuse_1206_3216Metric_Pad1.42x1.75mm_HandSolder, F.Cu at (193.5, 117.6)
- added J10: SM03B-SRSS-TB, Connector_JST:JST_SH_SM03B-SRSS-TB_1x03-1MP_P1.00mm_Horizontal, F.Cu at (257.2, 99.3)
- added J4: SM03B-SRSS-TB, Connector_JST:JST_SH_BM03B-SRSS-TB_1x03-1MP_P1.00mm_Vertical, F.Cu at (215.7, 132.5)
- added J5: SM03B-SRSS-TB, Connector_JST:JST_SH_SM03B-SRSS-TB_1x03-1MP_P1.00mm_Horizontal, F.Cu at (263.8, 40.7)
- added J6: SM03B-SRSS-TB, Connector_JST:JST_SH_BM03B-SRSS-TB_1x03-1MP_P1.00mm_Vertical, F.Cu at (122.0, 168.5)
- added J7: Conn_ARM_JTAG_SWD_10, Connector_PinHeader_1.27mm:PinHeader_2x05_P1.27mm_Vertical_SMD, F.Cu at (254.8, 57.0)
- added J8: Conn_ST_STDC14, Connector_PinHeader_1.27mm:PinHeader_2x07_P1.27mm_Vertical_SMD, F.Cu at (264.6, 57.5)
- added J9: SM03B-SRSS-TB, Connector_JST:JST_SH_SM03B-SRSS-TB_1x03-1MP_P1.00mm_Horizontal, F.Cu at (263.8, 48.3)
- added JP2: SolderJumper_2_Bridged, Jumper:SolderJumper-2_P1.3mm_Bridged_RoundedPad1.0x1.5mm, F.Cu at (173.7, 115.0)
- added JP3: SolderJumper_2_Bridged, Jumper:SolderJumper-2_P1.3mm_Bridged_RoundedPad1.0x1.5mm, F.Cu at (173.7, 118.5)
- added JP4: SolderJumper_2_Bridged, Jumper:SolderJumper-2_P1.3mm_Bridged_RoundedPad1.0x1.5mm, F.Cu at (173.7, 122.1)
- added JP5: SolderJumper_2_Bridged, Jumper:SolderJumper-2_P1.3mm_Bridged_RoundedPad1.0x1.5mm, F.Cu at (173.7, 125.6)
- added L1: 3.3u, ProjectSpecific:L_pol_2016, F.Cu at (117.5, 145.0)
- added L2: 3.3u, ProjectSpecific:L_pol_2016, F.Cu at (223.9, 123.8)
- added R50: 470R, Resistor_SMD:R_0402_1005Metric_Pad0.72x0.64mm_HandSolder, F.Cu at (97.5, 41.0)
- added R51: 470R, Resistor_SMD:R_0402_1005Metric_Pad0.72x0.64mm_HandSolder, F.Cu at (100.5, 41.0)
- added R52: 470R, Resistor_SMD:R_0402_1005Metric_Pad0.72x0.64mm_HandSolder, F.Cu at (62.5, 76.0)
- added R57: 1k, Resistor_SMD:R_0402_1005Metric, F.Cu at (225.4, 110.7)
- added R58: 1k, Resistor_SMD:R_0402_1005Metric, F.Cu at (98.5, 166.5)
- added R59: 1k, Resistor_SMD:R_0402_1005Metric, F.Cu at (116.0, 163.5)
- added R60: 33, Resistor_SMD:R_0402_1005Metric, F.Cu at (120.5, 145.5)
- added R61: 1k, Resistor_SMD:R_0402_1005Metric, F.Cu at (98.5, 163.5)
- added R62: 27, Resistor_SMD:R_0402_1005Metric, F.Cu at (114.5, 144.5)
- added R63: 27, Resistor_SMD:R_0402_1005Metric, F.Cu at (115.5, 144.5)
- added R64: 1k, Resistor_SMD:R_0402_1005Metric, F.Cu at (225.4, 112.7)
- added R65: 33, Resistor_SMD:R_0402_1005Metric, F.Cu at (225.4, 114.6)
- added R66: 1k, Resistor_SMD:R_0402_1005Metric, F.Cu at (225.4, 116.6)
- added R67: 27, Resistor_SMD:R_0402_1005Metric, F.Cu at (225.4, 118.6)
- added R68: 27, Resistor_SMD:R_0402_1005Metric, F.Cu at (225.4, 120.6)
- added R69: 100R, Resistor_SMD:R_0402_1005Metric_Pad0.72x0.64mm_HandSolder, F.Cu at (251.7, 37.9)
- added R70: 100R, Resistor_SMD:R_0402_1005Metric_Pad0.72x0.64mm_HandSolder, F.Cu at (251.7, 39.8)
- added R71: 100R, Resistor_SMD:R_0402_1005Metric_Pad0.72x0.64mm_HandSolder, F.Cu at (251.7, 41.8)
- added R72: 100R, Resistor_SMD:R_0402_1005Metric_Pad0.72x0.64mm_HandSolder, F.Cu at (251.7, 43.8)
- added R73: 100R, Resistor_SMD:R_0402_1005Metric_Pad0.72x0.64mm_HandSolder, F.Cu at (251.7, 45.8)
- added R74: 100R, Resistor_SMD:R_0402_1005Metric_Pad0.72x0.64mm_HandSolder, F.Cu at (251.7, 47.8)
- added R75: 100R, Resistor_SMD:R_0402_1005Metric_Pad0.72x0.64mm_HandSolder, F.Cu at (251.7, 49.8)
- added R76: 100R, Resistor_SMD:R_0402_1005Metric_Pad0.72x0.64mm_HandSolder, F.Cu at (251.7, 51.8)
- added R77: 100R, Resistor_SMD:R_0402_1005Metric_Pad0.72x0.64mm_HandSolder, F.Cu at (254.9, 37.9)
- added R78: 100R, Resistor_SMD:R_0402_1005Metric_Pad0.72x0.64mm_HandSolder, F.Cu at (254.9, 39.8)
- added R79: 100R, Resistor_SMD:R_0402_1005Metric_Pad0.72x0.64mm_HandSolder, F.Cu at (254.9, 41.8)
- added R80: 100R, Resistor_SMD:R_0402_1005Metric_Pad0.72x0.64mm_HandSolder, F.Cu at (254.9, 43.8)
- added R81: 100R, Resistor_SMD:R_0402_1005Metric_Pad0.72x0.64mm_HandSolder, F.Cu at (254.9, 45.8)
- added R82: 100R, Resistor_SMD:R_0402_1005Metric_Pad0.72x0.64mm_HandSolder, F.Cu at (254.9, 47.8)
- added R83: 100R, Resistor_SMD:R_0402_1005Metric_Pad0.72x0.64mm_HandSolder, F.Cu at (254.9, 49.8)
- added R84: 100R, Resistor_SMD:R_0402_1005Metric_Pad0.72x0.64mm_HandSolder, F.Cu at (254.9, 51.8)
- added R85: 100R, Resistor_SMD:R_0402_1005Metric_Pad0.72x0.64mm_HandSolder, F.Cu at (258.2, 37.9)
- added R86: 100R, Resistor_SMD:R_0402_1005Metric_Pad0.72x0.64mm_HandSolder, F.Cu at (258.2, 39.8)
- added R87: 100R, Resistor_SMD:R_0402_1005Metric_Pad0.72x0.64mm_HandSolder, F.Cu at (258.2, 41.8)
- added R88: 100R, Resistor_SMD:R_0402_1005Metric_Pad0.72x0.64mm_HandSolder, F.Cu at (258.2, 43.8)
- added R89: 100R, Resistor_SMD:R_0402_1005Metric_Pad0.72x0.64mm_HandSolder, F.Cu at (258.2, 45.8)
- added R90: 100R, Resistor_SMD:R_0402_1005Metric_Pad0.72x0.64mm_HandSolder, F.Cu at (258.2, 47.8)
- added R91: 100R, Resistor_SMD:R_0402_1005Metric_Pad0.72x0.64mm_HandSolder, F.Cu at (70.0, 37.5)
- added R92: 100R, Resistor_SMD:R_0402_1005Metric_Pad0.72x0.64mm_HandSolder, F.Cu at (251.7, 88.9)
- added R93: 100R, Resistor_SMD:R_0402_1005Metric_Pad0.72x0.64mm_HandSolder, F.Cu at (251.7, 90.9)
- added R94: 100R, Resistor_SMD:R_0402_1005Metric_Pad0.72x0.64mm_HandSolder, F.Cu at (251.7, 92.9)
- added R95: 100R, Resistor_SMD:R_0402_1005Metric_Pad0.72x0.64mm_HandSolder, F.Cu at (251.7, 94.9)
- added R96: 470R, Resistor_SMD:R_0402_1005Metric_Pad0.72x0.64mm_HandSolder, F.Cu at (251.7, 96.9)
- added R97: 470R, Resistor_SMD:R_0402_1005Metric_Pad0.72x0.64mm_HandSolder, F.Cu at (258.2, 49.8)
- added SW1: SW_Push, Button_Switch_SMD:SW_Push_1P1T_XKB_TS-1187A, F.Cu at (103.5, 161.5)
- added SW2: SW_Push, Button_Switch_SMD:SW_Push_1P1T_XKB_TS-1187A, F.Cu at (103.5, 168.2)
- added SW3: SW_Push, Button_Switch_SMD:SW_Push_1P1T_XKB_TS-1187A, F.Cu at (207.4, 126.8)
- added SW4: SW_Push, Button_Switch_SMD:SW_Push_1P1T_XKB_TS-1187A, F.Cu at (207.4, 133.4)
- added U10: SRV05-4, Package_TO_SOT_SMD:SOT-23-6, F.Cu at (273.6, 116.7)
- added U11: SRV05-4, Package_TO_SOT_SMD:SOT-23-6, F.Cu at (269.1, 72.0)
- added U12: RP2350_80QFN, ProjectSpecific:RP2350-QFN-80-1EP_10x10_P0.4mm_EP3.4x3.4mm_ThermalVias, F.Cu at (217.8, 115.7)
- added U13: RP2350_80QFN, ProjectSpecific:RP2350-QFN-80-1EP_10x10_P0.4mm_EP3.4x3.4mm_ThermalVias, F.Cu at (114.5, 154.5)
- added U14: ~, Connector_JST:JST_SH_SM04B-SRSS-TB_1x04-1MP_P1.00mm_Horizontal, F.Cu at (272.1, 40.7)
- added U15: AMS1117-3.3, Package_TO_SOT_SMD:SOT-223-3_TabPin2, F.Cu at (185.3, 123.9)
- added U16: W25Q128JVS, Package_SO:SOIC-8_5.3x5.3mm_P1.27mm, F.Cu at (108.5, 140.0)
- added U17: ~, Connector_JST:JST_SH_SM04B-SRSS-TB_1x04-1MP_P1.00mm_Horizontal, F.Cu at (257.7, 91.7)
- added U18: W25Q128JVS, Package_SO:SOIC-8_5.3x5.3mm_P1.27mm, F.Cu at (216.9, 125.2)
- added U8: INA219AxDCN, Package_TO_SOT_SMD:SOT-23-8, F.Cu at (273.6, 121.3)
- added U9: INA219AxDCN, Package_TO_SOT_SMD:SOT-23-8, F.Cu at (269.1, 76.7)
- added Y2: ABM8-272-T3, Crystal:Crystal_SMD_3225-4Pin_3.2x2.5mm, F.Cu at (115.5, 168.5)
- added Y3: ABM8-272-T3, Crystal:Crystal_SMD_3225-4Pin_3.2x2.5mm, F.Cu at (222.2, 130.9)
- A1: footprint Module:Arduino_UNO_R3 -> ProjectSpecific:Arduino_UNO_R3_ShieldBase
- C10, C5, C6, C7, C8, C9: footprint Capacitor_SMD:C_0402_1005Metric -> Capacitor_SMD:C_0402_1005Metric_Pad0.74x0.62mm_HandSolder
- JP1: footprint Jumper:SolderJumper-2_P1.3mm_Open_TrianglePad1.0x1.5mm -> Jumper:SolderJumper-2_P1.3mm_Open_RoundedPad1.0x1.5mm
- R16, R17, R18, R19, R20, R21, R22, R23, R24, R25, R26, R27, R28, R29, R30, R31, R39, R40, R41, R42, R43, R44, R45: value 470R -> 100R; footprint Resistor_SMD:R_0402_1005Metric -> Resistor_SMD:R_0402_1005Metric_Pad0.72x0.64mm_HandSolder
- R32, R33, R34, R35, R36, R37, R38, R46, R47, R48, R49: footprint Resistor_SMD:R_0402_1005Metric -> Resistor_SMD:R_0402_1005Metric_Pad0.72x0.64mm_HandSolder
- U1: value INA219AxDCN -> ~; footprint Package_TO_SOT_SMD:SOT-23-8 -> Connector_JST:JST_SH_SM04B-SRSS-TB_1x04-1MP_P1.00mm_Horizontal
- moved J2 225.1 mm to (262.8, 119.4), turned to 0 degrees
- moved J3 219.0 mm to (258.3, 74.8), turned to 0 degrees
- moved U7 214.4 mm to (269.1, 67.4)
- moved R12 214.2 mm to (268.0, 79.9)
- moved R15 214.2 mm to (268.0, 81.9)
- moved R14 207.3 mm to (261.9, 83.8)
- moved U6 206.9 mm to (273.6, 112.1)
- moved R11 205.6 mm to (272.5, 126.5)
- moved R8 204.9 mm to (272.5, 124.5)
- moved R13 203.2 mm to (257.7, 83.8)
- moved R10 200.3 mm to (266.3, 128.4)
- moved R9 199.6 mm to (262.1, 128.4)
- moved J1 152.9 mm to (181.7, 115.0), turned to 0 degrees
- moved U1 148.2 mm to (194.6, 123.5), turned to 0 degrees
- moved U2 147.3 mm to (197.0, 130.5), turned to 0 degrees
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Connections:
- net /usb-port/SHUNT.H renamed Net-(U6-Vout)
- net /usb-port/SHUNT.L renamed Net-(J2-VBUS)
- net /usb-port/~{EN} renamed /Tester/EN_USB_0
- net /usb-port/~{FLAG} renamed /Tester/FLAG_USB_0
- net /usb-port1/SHUNT.H renamed Net-(U7-Vout)
- net /usb-port1/SHUNT.L renamed Net-(J3-VBUS)
- net /usb-port1/~{EN} renamed /Tester/EN_USB_1
- net /usb-port1/~{FLAG} renamed /Tester/FLAG_USB_1
- A1 pad 10: /uno/A1 -> /Tester/uno/AI1
- A1 pad 11: /uno/A2 -> /Tester/uno/AI2
- A1 pad 12: /uno/A3 -> /Tester/uno/AI3
- A1 pad 13: /uno/A4 -> /Tester/uno/AI4
- A1 pad 14: /uno/A5 -> /Tester/uno/AI5
- A1 pad 3: /uno/~{RESET} -> Net-(A1-~{RESET})
- A1 pad 30: Net-(A1-AREF) -> /Tester/uno/AI6
- A1 pad 9: /uno/A0 -> /Tester/uno/AI0
- D1 pad 2: /USB/I2C.SDA -> /USB/LED4
- D2 pad 1: /USB/I2C.SDA -> /USB/LED4
- D3 pad 2: /USB/I2C.SDA -> /USB/LED4
- D4 pad 1: /USB/I2C.SDA -> /USB/LED4
- JP1 pad 1: Net-(A1-AREF) -> GND
- JP1 pad 2: +3V3 -> Net-(JP1-B)
- R16 pad 1: /uno/A0 -> /Tester/D0
- R16 pad 2: Net-(C5-Pad1) -> Net-(A1-D0/RX)
- R17 pad 1: /uno/D0 -> /Tester/D1
- R17 pad 2: Net-(A1-D0/RX) -> Net-(A1-D1/TX)
- R18 pad 1: /uno/D1 -> /Tester/D2
- R18 pad 2: Net-(A1-D1/TX) -> Net-(A1-D2)
- R19 pad 1: /uno/D2 -> /Tester/D3
- R19 pad 2: Net-(A1-D2) -> Net-(A1-D3)
- R20 pad 1: /uno/D3 -> /Tester/D4
- R20 pad 2: Net-(A1-D3) -> Net-(A1-D4)
- R21 pad 1: /uno/D4 -> /Tester/D5
- R21 pad 2: Net-(A1-D4) -> Net-(A1-D5)
- R22 pad 1: /uno/D5 -> /Tester/D6
- R22 pad 2: Net-(A1-D5) -> Net-(A1-D6)
- R23 pad 1: /uno/D6 -> /Tester/D7
- R23 pad 2: Net-(A1-D6) -> Net-(A1-D7)
- R24 pad 1: /uno/D7 -> /Tester/D8
- R24 pad 2: Net-(A1-D7) -> Net-(A1-D8)
- R25 pad 1: /uno/D8 -> /Tester/D9
- R25 pad 2: Net-(A1-D8) -> Net-(A1-D9)
- R26 pad 1: /uno/D9 -> /Tester/D10
- R26 pad 2: Net-(A1-D9) -> Net-(A1-D10)
- R27 pad 1: /uno/D10 -> /Tester/D11
- R27 pad 2: Net-(A1-D10) -> Net-(A1-D11)
- R28 pad 1: /uno/D11 -> /Tester/D12
- R28 pad 2: Net-(A1-D11) -> Net-(A1-D12)
- R29 pad 1: /uno/D12 -> /Tester/D13
- R29 pad 2: Net-(A1-D12) -> Net-(A1-D13)
- R30 pad 1: /uno/D13 -> Net-(A1-SDA/A4-Pad31)
- R30 pad 2: Net-(A1-D13) -> /Tester/D14
- R31 pad 1: /uno/A0 -> Net-(A1-SCL/A5-Pad32)
- R31 pad 2: /uno/A0 -> /Tester/D15
- R32 pad 1: /uno/A1 -> /Tester/uno/AI0
- R32 pad 2: /uno/A1 -> Net-(C5-Pad1)
- R33 pad 1: /uno/A2 -> /Tester/uno/AI1
- R33 pad 2: /uno/A2 -> Net-(C6-Pad1)
- R34 pad 1: /uno/A3 -> /Tester/uno/AI2
- R34 pad 2: /uno/A3 -> Net-(C7-Pad1)
- R35 pad 1: /uno/A4 -> /Tester/uno/AI3
- R35 pad 2: /uno/A4 -> Net-(C8-Pad1)
- R36 pad 1: /uno/A5 -> /Tester/uno/AI4
- R36 pad 2: /uno/A5 -> Net-(C9-Pad1)
- R37 pad 1: /uno/A1 -> /Tester/uno/AI5
- R37 pad 2: Net-(C6-Pad1) -> Net-(C10-Pad1)
- R38 pad 1: Net-(A1-SDA/A4-Pad31) -> /Tester/uno/AI6
- R38 pad 2: /uno/D14 -> Net-(C11-Pad1)
- R39 pad 1: Net-(A1-SCL/A5-Pad32) -> /Tester/uno/AI0
- R39 pad 2: /uno/D15 -> /Tester/A0
- R40 pad 1: /uno/A2 -> /Tester/uno/AI1
- R40 pad 2: Net-(C7-Pad1) -> /Tester/A1
- R41 pad 1: /uno/A3 -> /Tester/uno/AI2
- R41 pad 2: Net-(C8-Pad1) -> /Tester/A2
- R42 pad 1: /uno/A4 -> /Tester/uno/AI3
- R42 pad 2: Net-(C9-Pad1) -> /Tester/A3
- R43 pad 1: /uno/A5 -> /Tester/uno/AI4
- R43 pad 2: Net-(C10-Pad1) -> /Tester/A4
- R44 pad 1: Net-(C5-Pad1) -> /Tester/uno/AI5
- R44 pad 2: /uno/PWM0 -> /Tester/A5
- R45 pad 1: Net-(C6-Pad1) -> /Tester/uno/AI6
- R45 pad 2: /uno/PWM1 -> /Tester/A6
- R46 pad 1: Net-(C7-Pad1) -> Net-(C5-Pad1)
- R46 pad 2: /uno/PWM2 -> /Tester/PWM0
- R47 pad 1: Net-(C8-Pad1) -> Net-(C6-Pad1)
- R47 pad 2: /uno/PWM3 -> /Tester/PWM1
- R48 pad 1: Net-(C9-Pad1) -> Net-(C7-Pad1)
- R48 pad 2: /uno/PWM4 -> /Tester/PWM2
- R49 pad 1: Net-(C10-Pad1) -> Net-(C8-Pad1)
- R49 pad 2: /uno/PWM5 -> /Tester/PWM3
- R7 pad 1: /USB/I2C.SDA -> /USB/LED4
- U1 pad 1: unconnected-(U1-IN+-Pad1) -> /USB/SCL
- U1 pad 2: unconnected-(U1-IN--Pad2) -> /USB/SDA
- U1 pad 3: unconnected-(U1-GND-Pad3) -> Net-(JP5-A)
- U1 pad 4: unconnected-(U1-VS-Pad4) -> GND
- U3 pad 5: /USB/I2C.SDA -> /USB/SDA
- U3 pad 8: /USB/VDD33 -> Net-(JP5-A)
- U4 pad 13: /USB/I2C.SCL -> Net-(JP3-A)
- U4 pad 16: /USB/~{RESET} -> Net-(JP1-B)
- U4 pad 18: /USB/PSELF -> Net-(JP2-B)
- U4 pad 21: /USB/I2C.SDA -> /USB/LED4
- U4 pad 7: /USB/USB3.D+ -> /Tester/USB.D+
- U4 pad 8: /USB/USB3.D- -> /Tester/USB.D-

Commit message: Layout Tester and USB Hub
Parts:
- removed J8: Conn_ST_STDC14, Connector_PinHeader_1.27mm:PinHeader_2x07_P1.27mm_Vertical_SMD
- removed R75, R76, R77, R78, R79, R80, R82, R83, R84: 100R, Resistor_SMD:R_0402_1005Metric_Pad0.72x0.64mm_HandSolder
- added C58: 100nF, Capacitor_SMD:C_0402_1005Metric, F.Cu at (40.9, 57.0)
- added C59: 100nF, Capacitor_SMD:C_0402_1005Metric, F.Cu at (40.9, 72.0)
- U1: moved to B.Cu
- U4: footprint Package_DFN_QFN:QFN-24-1EP_4x4mm_P0.5mm_EP2.7x2.7mm -> Package_DFN_QFN:QFN-24-1EP_4x4mm_P0.5mm_EP2.7x2.7mm_ThermalVias
- moved R11 240.1 mm to (43.4, 54.5), turned to 180 degrees
- moved J2 239.0 mm to (30.9, 61.5), turned to -90 degrees
- moved U8 238.9 mm to (43.4, 57.5), turned to -90 degrees
- moved U10 237.7 mm to (42.4, 61.5)
- moved U6 232.7 mm to (47.9, 55.5)
- moved R8 232.7 mm to (49.4, 58.5), turned to 90 degrees
- moved R10 230.3 mm to (46.9, 58.5), turned to 180 degrees
- moved J3 227.4 mm to (30.9, 77.5), turned to -90 degrees
- moved U11 226.8 mm to (42.4, 77.5)
- moved U9 225.8 mm to (43.4, 73.0), turned to -90 degrees
- moved R15 224.4 mm to (43.9, 70.0), turned to 180 degrees
- moved R9 222.7 mm to (51.4, 56.5), turned to -90 degrees
- moved C13 222.3 mm to (43.9, 66.5), turned to 90 degrees
- moved U7 221.3 mm to (47.9, 72.0)
- moved R12 216.7 mm to (51.4, 73.0), turned to 180 degrees
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Connections:
- C4 pad 1: /USB/VDD33 -> Net-(JP5-A)
- U13 pad 42: /Tester/PWM0 -> /Tester/PWM6
- U13 pad 43: /Tester/PWM1 -> /Tester/PWM5
- U13 pad 44: /Tester/PWM2 -> /Tester/PWM4
- U13 pad 46: /Tester/PWM4 -> /Tester/PWM2
- U13 pad 47: /Tester/PWM5 -> /Tester/PWM1
- U13 pad 48: /Tester/PWM6 -> /Tester/PWM0
- U2 pad 1: /USB/D+ -> /USB/D-
- U2 pad 3: /USB/D- -> /USB/D+
- U2 pad 4: unconnected-(U2-IO3-Pad4) -> /USB/D+
- U2 pad 6: unconnected-(U2-IO4-Pad6) -> /USB/D-
- U4 pad 25: (no net) -> GND
Routing:
- net GND: track 0.00 -> 165.0 mm, vias 0 -> 65
- net /Tester/D13: track 0.00 -> 92.9 mm, vias 0 -> 3
- net +3V3: track 0.00 -> 86.9 mm, vias 0 -> 17
- net /Tester/D12: track 0.00 -> 85.7 mm, vias 0 -> 3
- net /Tester/D11: track 0.00 -> 77.0 mm, vias 0 -> 3
- net /Tester/D10: track 0.00 -> 69.5 mm, vias 0 -> 3
- net /Tester/~{TARGET_RESET}: track 0.00 -> 58.6 mm, vias 0 -> 2
- net /USB/USB2.D+: track 0.00 -> 57.6 mm, vias 0 -> 2
- net /USB/USB2.D-: track 0.00 -> 56.3 mm, vias 0 -> 2
- net /Tester/A6: track 0.00 -> 51.7 mm
- net /Tester/PWM6: track 0.00 -> 51.1 mm, vias 0 -> 2
- net /Tester/D15: track 0.00 -> 45.7 mm, vias 0 -> 2
- net /Tester/D14: track 0.00 -> 43.6 mm, vias 0 -> 2
- net Net-(J3-VBUS): track 0.00 -> 43.1 mm
- net /Tester/USB.D-: track 0.00 -> 41.7 mm, vias 0 -> 2
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- added copper zone on F.Cu, net +3V3
- added copper zone on In2.Cu, net +3V3
- added copper zone on In2.Cu, net +5V
- added copper zone on In2.Cu, net /Tester/RP2350B/+1V1
- added copper zone on F.Cu, net GND
- added copper zone on In1.Cu, net GND
Other:
- board outline added: 85.4 x 53.8 mm
- copper layers 2 -> 4

Commit message: WIP
Parts:
- removed C50, C51: 100nF, Capacitor_SMD:C_0402_1005Metric
- removed U16, U18: W25Q128JVS, Package_SO:SOIC-8_5.3x5.3mm_P1.27mm
- J10, J5, J9: value SM03B-SRSS-TB -> BM03B-SRSS-TB; footprint Connector_JST:JST_SH_SM03B-SRSS-TB_1x03-1MP_P1.00mm_Horizontal -> Connector_JST:JST_SH_BM03B-SRSS-TB_1x03-1MP_P1.00mm_Vertical
- J4, J6: value SM03B-SRSS-TB -> BM03B-SRSS-TB
- R57, R58, R59, R61, R64, R66: value 1k -> 1K
- U12, U13: value RP2350_80QFN -> RP2354B
- moved U14 149.7 mm to (64.5, 34.5), turned to 180 degrees
- moved J5 138.7 mm to (67.8, 60.7)
- moved R89 135.5 mm to (64.9, 39.4), turned to 90 degrees
- moved R90 134.5 mm to (66.0, 39.4), turned to 90 degrees
- moved R85 134.3 mm to (66.5, 56.0), turned to -90 degrees
- moved R81 132.9 mm to (65.5, 70.5)
- moved R86 131.6 mm to (69.0, 56.0), turned to -90 degrees
- moved R69 130.1 mm to (65.5, 65.2)
- moved J9 129.8 mm to (76.0, 60.7)
- moved J7 125.7 mm to (71.1, 67.7)
- moved R87 125.4 mm to (75.0, 56.1), turned to -90 degrees
- moved D7 123.4 mm to (88.3, 49.0), turned to 180 degrees
- moved R88 123.3 mm to (77.0, 56.1), turned to -90 degrees
- moved R70 119.6 mm to (77.0, 71.0), turned to 180 degrees
- moved R71 118.3 mm to (77.0, 66.5), turned to 180 degrees
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Connections:
- U12 pad 70: /debugger/RP2350B1/QSPI_SD3 -> unconnected-(U12-QSPI_SD3-Pad70)
- U12 pad 71: /debugger/RP2350B1/QSPI_SCLK -> unconnected-(U12-QSPI_SCLK-Pad71)
- U12 pad 72: /debugger/RP2350B1/QSPI_SD0 -> unconnected-(U12-QSPI_SD0-Pad72)
- U12 pad 73: /debugger/RP2350B1/QSPI_SD2 -> unconnected-(U12-QSPI_SD2-Pad73)
- U12 pad 74: /debugger/RP2350B1/QSPI_SD1 -> unconnected-(U12-QSPI_SD1-Pad74)
- U13 pad 70: /Tester/RP2350B/QSPI_SD3 -> unconnected-(U13-QSPI_SD3-Pad70)
- U13 pad 71: /Tester/RP2350B/QSPI_SCLK -> unconnected-(U13-QSPI_SCLK-Pad71)
- U13 pad 72: /Tester/RP2350B/QSPI_SD0 -> unconnected-(U13-QSPI_SD0-Pad72)
- U13 pad 73: /Tester/RP2350B/QSPI_SD2 -> unconnected-(U13-QSPI_SD2-Pad73)
- U13 pad 74: /Tester/RP2350B/QSPI_SD1 -> unconnected-(U13-QSPI_SD1-Pad74)
Routing:
- net /Tester/RP2350B/QSPI_SS: track 25.1 -> 3.77 mm
- net /Tester/RP2350B/QSPI_SD1: track 20.3 -> 0.00 mm
- net /Tester/RP2350B/QSPI_SD2: track 15.9 -> 0.00 mm
- net /Tester/RP2350B/QSPI_SD3: track 14.1 -> 0.00 mm
- net /Tester/RP2350B/QSPI_SCLK: track 12.7 -> 0.00 mm
- net /Tester/RP2350B/QSPI_SD0: track 10.3 -> 0.00 mm
- net /Tester/A6: track 51.7 -> 57.5 mm, vias 0 -> 2
- net /Tester/PWM6: track 51.1 -> 56.7 mm
- net GND: track 165.0 -> 160.3 mm, vias 65 -> 67
- net Net-(A1-D0/RX): track 0.00 -> 3.63 mm
- net +3V3: track 86.9 -> 83.5 mm, vias 17 -> 16
- net Net-(J10-Pin_1): track 3.85 -> 7.17 mm
- net Net-(J10-Pin_3): track 3.06 -> 6.39 mm
- net Net-(A1-D1/TX): track 0.00 -> 3.13 mm
- net Net-(A1-D2): track 0.00 -> 2.66 mm
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- added copper zone on B.Cu, net +3V3
- added copper zone on In1.Cu, net +3V3
- added copper zone on In1.Cu, net +5V
- added copper zone on B.Cu, net /Tester/RP2350B/+1V1
- added copper zone on In2.Cu, net GND
- removed copper zone on F.Cu, net +3V3
- removed copper zone on In2.Cu, net +3V3
- removed copper zone on In2.Cu, net +5V
- removed copper zone on In2.Cu, net /Tester/RP2350B/+1V1
- removed copper zone on In1.Cu, net GND
Other:
- outline, holes or cut-outs redrawn

Commit message: finished routing
Parts:
- moved R70 11.5 mm to (65.5, 71.8), turned to 0 degrees
- moved C2 6.52 mm to (49.3, 45.7)
- moved C3 6.52 mm to (50.3, 45.7)
- moved C56 6.52 mm to (53.3, 62.6)
- moved R3 6.52 mm to (56.8, 33.6)
- moved U5 6.52 mm to (56.8, 36.6)
- moved C1 6.52 mm to (53.7, 35.0)
- moved C12 6.52 mm to (59.9, 42.4)
- moved C13 6.52 mm to (50.4, 66.5)
- moved C4 6.52 mm to (41.9, 51.0)
- moved C52 6.52 mm to (48.4, 82.0)
- moved C53 6.52 mm to (48.0, 34.5)
- moved C54 6.52 mm to (51.0, 34.5)
- moved C55 6.52 mm to (48.0, 44.2)
- moved C57 6.52 mm to (58.7, 59.2)
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Routing:
- net /Tester/I2C.SCL: track 0.00 -> 112.0 mm, vias 0 -> 3
- net /Tester/I2C.SDA: track 0.00 -> 108.1 mm, vias 0 -> 3
- net /Tester/FLAG_USB_0: track 6.37 -> 78.7 mm, vias 1 -> 3
- net /Tester/EN_USB_0: track 3.26 -> 64.1 mm, vias 1 -> 3
- net /Tester/EN_USB_1: track 5.38 -> 62.6 mm, vias 1 -> 2
- net /Tester/FLAG_USB_1: track 5.22 -> 60.5 mm, vias 1 -> 2
- net +3V3: track 83.5 -> 133.3 mm, vias 16 -> 33
- net GND: track 160.3 -> 209.5 mm, vias 67 -> 100
- net /debugger/Vref: track 0.00 -> 45.2 mm, vias 0 -> 2
- net /Tester/SWD.SWCLK: track 13.0 -> 51.5 mm, vias 0 -> 2
- net /Tester/TODI: track 0.00 -> 36.6 mm, vias 0 -> 2
- net /Tester/TIDO: track 0.00 -> 35.2 mm, vias 0 -> 2
- net /Tester/SWD.SWD: track 11.0 -> 45.4 mm, vias 0 -> 2
- net /debugger/SWCLK: track 0.00 -> 33.2 mm, vias 0 -> 2
- net /debugger/~{TARGET_RESET}: track 0.00 -> 31.9 mm, vias 0 -> 2
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- added copper zone on B.Cu, net /debugger/RP2350B1/+1V1
Other:
- board size 85.4 x 53.8 mm -> 78.9 x 53.8 mm

Commit message: layout finished
Parts:
- U1: moved to F.Cu
- U12, U13: footprint ProjectSpecific:RP2350-QFN-80-1EP_10x10_P0.4mm_EP3.4x3.4mm_ThermalVias -> Package_DFN_QFN:QFN-80-1EP_10x10mm_P0.4mm_EP3.4x3.4mm_ThermalVias
- moved JP5 15.3 mm to (54.2, 52.5), turned to 0 degrees
- moved C4 9.69 mm to (51.5, 52.4)
- moved R7 4.18 mm to (61.6, 52.5)
- moved D5 4.13 mm to (59.3, 52.5)
- moved JP3 2.18 mm to (41.1, 50.0)
- moved JP4 2.18 mm to (41.1, 47.5)
- moved U1 0.49 mm to (35.6, 49.8), turned to -90 degrees
- moved D1 0.09 mm to (52.7, 48.1)
- moved D3 0.09 mm to (56.3, 48.1)
Routing:
- net +3V3: track 133.3 -> 153.4 mm, vias 33 -> 34
- net /USB/VDD33: track 28.5 -> 17.8 mm
- net Net-(JP5-A): track 9.86 -> 17.2 mm, vias 1 -> 0
- net GND: track 209.5 -> 212.1 mm
- net Net-(JP3-A): track 20.9 -> 18.5 mm
- net /debugger/RP2350B1/+1V1: track 16.3 -> 17.9 mm, vias 4 -> 6
- net /USB/SCL: track 8.38 -> 7.79 mm, vias 1 -> 0
- net /USB/SDA: track 14.8 -> 14.4 mm, vias 1 -> 0
Other:
- board text added: "A"
- board text added: "A T B D"
- board text added: "A0"
- board text added: "A5"
- board text added: "B"
- board text added: "CH334"
- board text added: "CH334 EEPROM Qwicc"
- board text added: "D Boot"
- board text added: "D Reset"
- board text added: "D0"
- board text added: "D13"
- board text added: "D14"
- board text added: "D8"
- board text added: "Debugger"
- board text added: "Debugger JTAG"
- board text added: "Debugger Qwicc"
- board text added: "G"
- board text added: "Ref"
- board text added: "Reset"
- board text added: "T Boot"
- board text added: "T Reset"
- board text added: "Target JTAG"
- board text added: "Target SWD"
- board text added: "Target UART"
- board text added: "Tester"
- board text added: "Tester JTAG"
- board text added: "Tester Qwicc"
- board text added: "Tester UART"
