File: shield.kicad_pcb (KiCad board)
At the start: 4 copper layers, 78.9 x 53.8 mm, 196 parts, among them J1 USB_C_Receptacle_USB2.0_16P, J2 USB_A, J3 USB_A, J4 BM03B-SRSS-TB, J5 BM03B-SRSS-TB, J6 BM03B-SRSS-TB, J7 Conn_ARM_JTAG_SWD_10, J9 BM03B-SRSS-TB, SW1 SW_Push, SW2 SW_Push, SW3 SW_Push, SW4 SW_Push, U1 StemmaQt, U10 SRV05-4, U11 SRV05-4, U12 RP2354B, U13 RP2354B, U14 StemmaQt, U15 AMS1117-3.3, U16 FSUSB42MUX, U17 StemmaQt, U2 SRV05-4, U3 M24C02-WMN, U4 CH334F, U5 CH217K, U6 CH217K, U7 CH217K, U8 INA219AxDCN, U9 INA219AxDCN, Y1 12Mhz, Y2 ABM8-272-T3, Y3 ABM8-272-T3

Commit message: Add mounting holes
Parts:
- added H1: MountingHole_Pad, MountingHole:MountingHole_2.5mm_Pad_Via, F.Cu at (87.9, 28.0)
- added H1: MountingHole_Pad, MountingHole:MountingHole_2.5mm_Pad_Via, F.Cu at (37.9, 28.0)
- added H3: MountingHole_Pad, MountingHole:MountingHole_2.5mm_Pad_Via, F.Cu at (47.9, 88.0)
- added H3: MountingHole_Pad, MountingHole:MountingHole_2.5mm_Pad_Via, F.Cu at (97.9, 88.0)
Routing:
- net (no net): vias 0 -> 1
Other:
- board size 78.9 x 53.8 mm -> 78.9 x 66 mm
