File: tester.kicad_sch (KiCad schematic)
At the start: 6 parts, among them J10 SM03B-SRSS-TB

Commit message: Start Layout
Parts:
- added D6: LED, LED_SMD:LED_0805_2012Metric, symbol Device:LED
- added R96: 470R, Resistor_SMD:R_0402_1005Metric_Pad0.72x0.64mm_HandSolder, symbol Device:R
- U17: symbol Project_Specific:StemmaQtTarget -> Project_Specific:StemmaQtController
Connections:
- net GND: now also R96.1
- new net: D6.1 (K), R96.2
- new net RP2350B/GPIO47: D6.2 (A)
Other:
- sheet uno ports: added none; removed IOREF

Commit message: Layout Tester and USB Hub
Changed lines of the file:
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@@
 		)
 	)
-	(label "PWM2"
+	(label "PWM4"
 		(at 91.44 120.65 180)
 		(effects
@@
 		)
 	)
-	(label "PWM0"
+	(label "PWM6"
 		(at 91.44 115.57 180)
 		(effects
@@
 		)
 	)
-	(label "PWM6"
+	(label "PWM0"
 		(at 91.44 130.81 180)
 		(effects
@@
 		)
 	)
-	(label "PWM1"
+	(label "PWM5"
 		(at 91.44 118.11 180)
 		(effects
@@
 		)
 	)
-	(label "PWM4"
+	(label "PWM2"
 		(at 91.44 125.73 180)
 		(effects
@@
 		)
 	)
-	(label "PWM5"
+	(label "PWM1"
 		(at 91.44 128.27 180)
 		(effects

Commit message: WIP
Parts:
- J10: value SM03B-SRSS-TB -> BM03B-SRSS-TB; footprint Connector_JST:JST_SH_SM03B-SRSS-TB_1x03-1MP_P1.00mm_Horizontal -> Connector_JST:JST_SH_BM03B-SRSS-TB_1x03-1MP_P1.00mm_Vertical; LCSC (none) -> C160389
Changed lines of the file:
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@@
 			)
 		)
-		(property "Value" "SM03B-SRSS-TB"
+		(property "Value" "BM03B-SRSS-TB"
 			(at 204.47 119.38 0)
 			(effects
@@
 			)
 		)
-		(property "Footprint" "Connector_JST:JST_SH_SM03B-SRSS-TB_1x03-1MP_P1.00mm_Horizontal"
+		(property "Footprint" "Connector_JST:JST_SH_BM03B-SRSS-TB_1x03-1MP_P1.00mm_Vertical"
 			(at 201.93 118.11 0)
 			(effects
@@
 			(at 201.93 118.11 0)
 			(effects
+				(font
+					(size 1.27 1.27)
+				)
+				(hide yes)
+			)
+		)
+		(property "LCSC" "C160389"
+			(at 201.93 118.11 0)
+			(effects

Commit message: JLC rotations
Parts:
- J10: FT Rotation Offset (none) -> 180
Changed lines of the file:
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@@
+			)
+		)
+		(property "FT Rotation Offset" ""
+			(at 189.23 115.57 90)
+			(effects
+				(font
+					(size 1.27 1.27)
+				)
+				(hide yes)
 			)
 		)
@@
 			)
 		)
+		(property "FT Rotation Offset" "180"
+			(at 201.93 118.11 0)
+			(effects
+				(font
+					(size 1.27 1.27)
+				)
+				(hide yes)
+			)
+		)
 		(pin "1"
 		)
@@
 			)
 		)
+		(property "FT Rotation Offset" ""
+			(at 87.63 173.99 90)
+			(effects
+				(font
+					(size 1.27 1.27)
+				)
+				(hide yes)
+			)
+		)
 		(pin "1"
 		)
@@
 			)
 		)
+		(property "FT Rotation Offset" ""
+			(at 201.93 86.36 0)
+			(effects
+				(font
+					(size 1.27 1.27)
+				)
+				(hide yes)
+			)
+		)
 		(pin "1"
 		)
@@
 			)
 		)
+		(property "FT Rotation Offset" ""
+			(at 87.63 163.83 0)
+			(effects
+				(font
+					(size 1.27 1.27)
+				)
+				(hide yes)
+			)
+		)
 		(pin "1"
 		)
@@
 			)
 		)
+		(property "FT Rotation Offset" ""
+			(at 189.23 120.65 90)
+			(effects
+				(font
+					(size 1.27 1.27)
+				)
+				(hide yes)
+			)
+		)
 		(pin "1"
 		)
@@
 			)
 		)
+		(property "FT Rotation Offset" ""
+			(at 187.96 85.09 90)
+			(effects
+				(font
+					(size 1.27 1.27)
+				)
+				(hide yes)
+			)
+		)
 		(pin "1"
 		)
@@
 			(at 187.96 87.63 90)
 			(effects
+				(font
+					(size 1.27 1.27)
+				)
+				(hide yes)
+			)
+		)
+		(property "FT Rotation Offset" ""
+			(at 187.96 87.63 90)
+			(effects

Commit message: Fix rev1 errors
Add USB mux to allow for USB PIO
Fix D+ D- mixup
Fix USB Hub LED indicator label
Parts:
- removed J10: BM03B-SRSS-TB, Connector_JST:JST_SH_BM03B-SRSS-TB_1x03-1MP_P1.00mm_Vertical, symbol Connector_Generic_MountingPin:Conn_01x03_MountingPin
- removed R94, R95: 100R, Resistor_SMD:R_0402_1005Metric_Pad0.72x0.64mm_HandSolder, symbol Device:R
- added R53, R54: 27, Resistor_SMD:R_0402_1005Metric, symbol Device:R
Connections:
- net SCL is gone; now on net I2C.SCL: R93.1
- net SDA is gone; now on net I2C.SDA: R92.1
- new net HD+: R53.2
- new net HD-: R54.2
- new net USBH.D+: R53.1
- new net USBH.D-: R54.1
Other:
- note removed: "JST UART Connector"

Commit message: Address board review comments
- Add pull-ups for both I2C busses (4K7)
- Set eFuse limit to 600mA (400mA before)
- Label StemmaQt as such in schematics
- Fix typo in USB Port value
- Fix USB Mux to be disabled by default (pull-down to pull-up)
Parts:
- added R75, R76: 4K7, Resistor_SMD:R_0402_1005Metric_Pad0.72x0.64mm_HandSolder, symbol Device:R
- U17: value ~ -> StemmaQt
Connections:
- net +3V3: now also R75.2, R76.2
- net I2C.SCL: now also R76.1
- net I2C.SDA: now also R75.1
