File: usb.kicad_sch (KiCad schematic)
At the start: 36 parts, among them J1 USB_C_Receptacle_USB2.0_14P, U15 AMS1117-3.3, U2 SRV05-4, U3 M24C02-WMN, U4 CH334F, U5 CH217K, Y1 12Mhz

Commit message: Address board review comments
- Add pull-ups for both I2C busses (4K7)
- Set eFuse limit to 600mA (400mA before)
- Label StemmaQt as such in schematics
- Fix typo in USB Port value
- Fix USB Mux to be disabled by default (pull-down to pull-up)
Parts:
- added R77, R78: 4K7, Resistor_SMD:R_0402_1005Metric_Pad0.72x0.64mm_HandSolder, symbol Device:R
- J1: value USB_C_Receptacle_USB2.0_14P -> USB_C_Receptacle_USB2.0_16P
- R3: value 150K -> 100K; LCSC C22807 -> C23162
- U1: value ~ -> StemmaQt
Connections:
- net SCL: now also R78.1
- net SDA: now also R77.1
- net at C4.1, JP5.1 (A), U1.3 (V+)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: now also R77.2, R78.2
Other:
- note added: "Iset=60K/R = 0.6A"
- note removed: "Iset=60K/R = 0.4A"
