File: shield.kicad_sch (KiCad schematic)
At the start: 0 parts

Commit message: Add mounting holes
Parts:
- added H1, H2, H3, H4: MountingHole_Pad, MountingHole:MountingHole_2.5mm_Pad_Via, symbol Mechanical:MountingHole_Pad
Connections:
- net GND: now also H1.1, H2.1, H3.1, H4.1
